Commit message: Run a single episode to generate a visualization graph, weights need to be adjusted, no self-collision evaluation.

File: data/urdf/rm_65_b_description/urdf/rm_65_b_description.urdf (robot description, URDF)
Before this commit: robot rm_65_b_description, 7 links, 6 joints
Joints:
- joint joint1: origin xyz=0 0 0.2405 rpy=0 0 0 -> xyz=0 0 0.2875 rpy=0 0 0

Commit message: New posture capability evaluation metrics and new visualization methods have been added.

File: data/urdf/rm_65_b_description/urdf/rm_65_b_description.urdf (robot description, URDF)
Before this commit: robot rm_65_b_description, 7 links, 6 joints
Joints:
- joint joint1: origin xyz=0 0 0.2875 rpy=0 0 0 -> xyz=0 0 0.2405 rpy=0 0 0
