Commit message: Voxelized orientation data mining

File: src/robots/realman/rm_description/urdf/rm_65.urdf (robot description, URDF)
Before this commit: robot rm_65_description, 7 links, 6 joints
Links:
- link Link1: geometry collision mesh filename=package://rm_description/meshes/rm_65_arm/link1.STL; visual mesh filename=package://rm_description/meshes/rm_65_arm/link1.STL
- link Link2: geometry collision mesh filename=package://rm_description/meshes/rm_65_arm/link2.STL; visual mesh filename=package://rm_description/meshes/rm_65_arm/link2.STL
- link Link3: geometry collision mesh filename=package://rm_description/meshes/rm_65_arm/link3.STL; visual mesh filename=package://rm_description/meshes/rm_65_arm/link3.STL
- link Link4: geometry collision mesh filename=package://rm_description/meshes/rm_65_arm/link4.STL; visual mesh filename=package://rm_description/meshes/rm_65_arm/link4.STL
- link Link5: geometry collision mesh filename=package://rm_description/meshes/rm_65_arm/link5.STL; visual mesh filename=package://rm_description/meshes/rm_65_arm/link5.STL
- link Link6: geometry collision mesh filename=package://rm_description/meshes/rm_65_arm/link6.STL; visual mesh filename=package://rm_description/meshes/rm_65_arm/link6.STL
- link base_link: geometry collision mesh filename=package://rm_description/meshes/rm_65_arm/base_link.STL; visual mesh filename=package://rm_description/meshes/rm_65_arm/base_link.STL
